File: Hardware/Panel/precadsr_panel_al/precadsr_panel_al.kicad_pcb (KiCad board)
At the start: 2 copper layers, 50 x 200 mm, 16 parts

Commit message: NPTH new version
Parts:
- added GP1: Ground_point_for_NPTH, Kosmo_panel:Ground_point_for_NPTH, F.Cu at (35.0, 155.0)
- H1, H2: footprint Kosmo_panel:Kosmo_Panel_Dual_Slotted_Mounting_Hole_NPTH -> Kosmo_panel:Kosmo_Panel_Dual_Slotted_Mounting_Holes_NPTH
Connections:
- H10 pad 1: (no net) -> GND
- H12 pad 1: (no net) -> GND
- H13 pad 1: (no net) -> GND
- H3 pad 1: (no net) -> GND
- H4 pad 1: (no net) -> GND
- H5 pad 1: (no net) -> GND
- H6 pad 1: (no net) -> GND
- H7 pad 1: (no net) -> GND
- H8 pad 1: (no net) -> GND
- H9 pad 1: (no net) -> GND
Routing:
- removed copper zone on B.Cu, net GND
